File: Design/COOF-80/COOF-80.kicad_sch (KiCad schematic)
At the start: 63 parts

Commit message: Fixes to schematic
+ Added taps/jumpers to system clock divider
+ Fixed UART wiring
Connections:
- net at U?.15 (~{BAUDOUT}): now also U?.9 (RCLK)
- net ~{CTS}: now reaches U?.36 (~{CTS})
- net ~{DTR}: no longer names the net of U?.33 (~{DTR})
Other:
- title: (none) -> COOF-80
Changed lines of the file:
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@@
 (kicad_sch (version 20211123) (generator eeschema)
   (paper "B")
+  (title_block
+    (title "COOF-80")
+    (date "2023-03-05")
+    (rev "A")
+  )
   (junction (at 210.82 107.95) (diameter 0) (color 0 0 0 0)
   )
@@
     (stroke (width 0) (type default) (color 0 0 0 0))
   )
+  (wire (pts (xy 402.59 115.57) (xy 403.86 115.57))
+    (stroke (width 0) (type default) (color 0 0 0 0))
+  )
   (wire (pts (xy 134.62 81.28) (xy 132.08 81.28))
     (stroke (width 0) (type default) (color 0 0 0 0))
@@
     (stroke (width 0) (type default) (color 0 0 0 0))
   )
+  (wire (pts (xy 402.59 110.49) (xy 403.86 110.49))
+    (stroke (width 0) (type default) (color 0 0 0 0))
+  )
   (wire (pts (xy 35.56 212.09) (xy 36.83 212.09))
     (stroke (width 0) (type default) (color 0 0 0 0))
@@
     (stroke (width 0) (type default) (color 0 0 0 0))
   )
+  (wire (pts (xy 402.59 57.15) (xy 407.67 57.15))
+    (stroke (width 0) (type default) (color 0 0 0 0))
+  )
   (wire (pts (xy 350.52 105.41) (xy 351.79 105.41))
     (stroke (width 0) (type default) (color 0 0 0 0))
@@
     (stroke (width 0) (type default) (color 0 0 0 0))
   )
-  (wire (pts (xy 402.59 67.31) (xy 407.67 67.31))
-    (stroke (width 0) (type default) (color 0 0 0 0))
-  )
   (wire (pts (xy 223.52 181.61) (xy 223.52 182.88))
     (stroke (width 0) (type default) (color 0 0 0 0))
@@
   )
   (wire (pts (xy 160.02 76.2) (xy 162.56 76.2))
+    (stroke (width 0) (type default) (color 0 0 0 0))
+  )
+  (wire (pts (xy 403.86 110.49) (xy 403.86 115.57))
     (stroke (width 0) (type default) (color 0 0 0 0))
   )
@@
     )
   )
-  (global_label "~{DTR}" (shape output) (at 407.67 67.31 0) (fields_autoplaced)
-    (effects (font (size 1.27 1.27)) (justify left))
-    (property "Intersheet References" "${INTERSHEET_REFS}" (id 0) (at 413.5907 67.2306 0)
-      (effects (font (size 1.27 1.27)) (justify left) hide)
-    )
-  )
   (global_label "~{CSRAM2}" (shape input) (at 245.11 158.75 180) (fields_autoplaced)
     (effects (font (size 1.27 1.27)) (justify right))
@@
     )
   )
+  (global_label "~{CTS}" (shape output) (at 407.67 57.15 0) (fields_autoplaced)
+    (effects (font (size 1.27 1.27)) (justify left))
+    (property "Intersheet References" "${INTERSHEET_REFS}" (id 0) (at 413.5302 57.0706 0)
+      (effects (font (size 1.27 1.27)) (justify left) hide)
+    )
+  )
